Commit message: removed is_connected to only be used in serial port, cleaned up functions and main paxi_hardware, added imu

File: paxi_ws/src/paxi_description/urdf/include/paxi_imu.xacro (robot description, xacro)
@@ -1,8 +1,10 @@
 <?xml version="1.0"?>
 <robot name="paxi_bot" xmlns:xacro="http://www.ros.org/wiki/xacro">
+    <xacro:property name="imu_joint_name" value="imu_joint"/>
+    <xacro:property name="imu_link_name" value="imu"/>
     <xacro:property name="imu_width" value="0.15"/>
     <xacro:property name="imu_length" value="0.05"/>
     <xacro:property name="imu_height" value="0.05"/>
-    //should be inside base box;
+    <!-- should be "inside base box"; -->
     <xacro:property name="imu_joint_offset_x" value="0.0"/>
     <xacro:property name="imu_joint_offset_y" value="0.0"/>

File: paxi_ws/src/paxi_description/urdf/paxi_bot.urdf (robot description, URDF)
Before this commit: robot paxi_bot, 9 links, 8 joints
Links:
- removed link {$imu_link_name}
- added link ${imu_link_name}; visual box size=${imu_length} ${imu_width} ${imu_height}
Joints:
- joint ${imu_joint_name}: origin xyz=${imu_joint_offset_x} ${lidar_box_joint_offset_y} ${lidar_box_joint_offset_z} rpy=0 0 0 -> xyz=${imu_joint_offset_x} ${imu_joint_offset_y} ${imu_joint_offset_z} rpy=0 0 0

Commit message: Ekf tweaing, and adding imu_slamtec_to urdf

File: paxi_ws/src/paxi_description/urdf/include/paxi_imu.xacro (robot description, xacro)
@@ -1,12 +1,12 @@
 <?xml version="1.0"?>
 <robot name="paxi_bot" xmlns:xacro="http://www.ros.org/wiki/xacro">
-    <xacro:property name="imu_joint_name" value="imu_joint"/>
-    <xacro:property name="imu_link_name" value="imu"/>
+    <xacro:property name="imu_joint_name" value="imu_slamtec_joint"/>
+    <xacro:property name="imu_link_name" value="imu_slamtec"/>
     <xacro:property name="imu_width" value="0.06"/>
     <xacro:property name="imu_length" value="0.15"/>
     <xacro:property name="imu_height" value="0.045"/>
     <!-- should be "inside base box"; -->
-    <xacro:property name="imu_joint_offset_x" value="0.0"/>
-    <xacro:property name="imu_joint_offset_y" value="0.20"/>
+    <xacro:property name="imu_joint_offset_x" value="0.3"/>
+    <xacro:property name="imu_joint_offset_y" value="0.0"/>
     <xacro:property name="imu_joint_offset_z" value="${base_height}"/>
 </robot>

File: paxi_ws/src/paxi_description/urdf/paxi_bot.urdf (robot description, URDF)
Before this commit: robot paxi_bot, 9 links, 8 joints
Links:
- added link ${imu_slamtec_link_name}; visual box size=${imu_slamtec_length} ${imu_slamtec_width} ${imu_slamtec_he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
Joints:
- added joint ${imu_slamtec_joint_name}: type fixed, parent base_box, child ${imu_slamtec_link_name}, origin xyz=${imu_slamtec_joint_offset_x} ${imu_slamtec_joint_offset_y} ${imu_slamtec_joint_offset_z} rpy=0 0 0

Commit message: Finalized imu_slamtec on URDF, updated launch file for correct frame

File: paxi_ws/src/paxi_description/urdf/include/paxi_imu.xacro (robot description, xacro)
@@ -1,12 +1,12 @@
 <?xml version="1.0"?>
 <robot name="paxi_bot" xmlns:xacro="http://www.ros.org/wiki/xacro">
-    <xacro:property name="imu_joint_name" value="imu_slamtec_joint"/>
-    <xacro:property name="imu_link_name" value="imu_slamtec"/>
+    <xacro:property name="imu_joint_name" value="imu_joint"/>
+    <xacro:property name="imu_link_name" value="imu"/>
     <xacro:property name="imu_width" value="0.06"/>
     <xacro:property name="imu_length" value="0.15"/>
     <xacro:property name="imu_height" value="0.045"/>
     <!-- should be "inside base box"; -->
-    <xacro:property name="imu_joint_offset_x" value="0.3"/>
-    <xacro:property name="imu_joint_offset_y" value="0.0"/>
+    <xacro:property name="imu_joint_offset_x" value="0.0"/>
+    <xacro:property name="imu_joint_offset_y" value="0.2"/>
     <xacro:property name="imu_joint_offset_z" value="${base_height}"/>
 </robot>

File: paxi_ws/src/paxi_description/urdf/include/paxi_imu_slamtec.xacro (robot description, xacro)
@@ -1,12 +1,12 @@
 <?xml version="1.0"?>
 <robot name="paxi_bot" xmlns:xacro="http://www.ros.org/wiki/xacro">
-    <xacro:property name="imu_slamtec_joint_name" value="imu_joint"/>
-    <xacro:property name="imu_slamtec_link_name" value="imu"/>
-    <xacro:property name="imu_slamtec_width" value="0.06"/>
-    <xacro:property name="imu_slamtec_length" value="0.15"/>
-    <xacro:property name="imu_slamtec_height" value="0.045"/>
+    <xacro:property name="imu_slamtec_joint_name" value="imu_slamtec_joint"/>
+    <xacro:property name="imu_slamtec_link_name" value="imu_slamtec"/>
+    <xacro:property name="imu_slamtec_width" value="0.0488"/>
+    <xacro:property name="imu_slamtec_length" value="0.0538"/>
+    <xacro:property name="imu_slamtec_height" value="0.0252"/>
     <!-- should be "inside base box"; -->
-    <xacro:property name="imu_slamtec_joint_offset_x" value="0.0"/>
-    <xacro:property name="imu_slamtec_joint_offset_y" value="0.4"/>
+    <xacro:property name="imu_slamtec_joint_offset_x" value="0.3"/>
+    <xacro:property name="imu_slamtec_joint_offset_y" value="0.0"/>
     <xacro:property name="imu_slamtec_joint_offset_z" value="${base_height}"/>
 </robot>

File: paxi_ws/src/paxi_description/urdf/paxi_bot.urdf (robot description, URDF)
Before this commit: robot paxi_bot, 10 links, 9 joints
Joints:
- joint ${imu_slamtec_joint_name}: parent base_box -> base_link

Commit message: Updated frane ID for slamtec to IMU, and hover to imu_hover

File: paxi_ws/src/paxi_description/urdf/include/paxi_imu.xacro (robot description, xacro)
@@ -2,5 +2,5 @@
 <robot name="paxi_bot" xmlns:xacro="http://www.ros.org/wiki/xacro">
     <xacro:property name="imu_joint_name" value="imu_joint"/>
-    <xacro:property name="imu_link_name" value="imu"/>
+    <xacro:property name="imu_link_name" value="imu_hover"/>
     <xacro:property name="imu_width" value="0.06"/>
     <xacro:property name="imu_length" value="0.15"/>

File: paxi_ws/src/paxi_description/urdf/include/paxi_imu_slamtec.xacro (robot description, xacro)
@@ -2,5 +2,5 @@
 <robot name="paxi_bot" xmlns:xacro="http://www.ros.org/wiki/xacro">
     <xacro:property name="imu_slamtec_joint_name" value="imu_slamtec_joint"/>
-    <xacro:property name="imu_slamtec_link_name" value="imu_slamtec"/>
+    <xacro:property name="imu_slamtec_link_name" value="imu"/>
     <xacro:property name="imu_slamtec_width" value="0.0488"/>
     <xacro:property name="imu_slamtec_length" value="0.0538"/>

Commit message: Added correct joing names and location of IMU

File: paxi_ws/src/paxi_description/urdf/include/paxi_imu.xacro (robot description, xacro)
@@ -7,6 +7,6 @@
     <xacro:property name="imu_height" value="0.045"/>
     <!-- should be "inside base box"; -->
-    <xacro:property name="imu_joint_offset_x" value="0.0"/>
-    <xacro:property name="imu_joint_offset_y" value="0.2"/>
+    <xacro:property name="imu_joint_offset_x" value="0.2"/>
+    <xacro:property name="imu_joint_offset_y" value="0.0"/>
     <xacro:property name="imu_joint_offset_z" value="${base_height}"/>
 </robot>

File: paxi_ws/src/paxi_description/urdf/include/paxi_imu_slamtec.xacro (robot description, xacro)
@@ -7,6 +7,6 @@
     <xacro:property name="imu_slamtec_height" value="0.0252"/>
     <!-- should be "inside base box"; -->
-    <xacro:property name="imu_slamtec_joint_offset_x" value="0.3"/>
-    <xacro:property name="imu_slamtec_joint_offset_y" value="0.0"/>
+    <xacro:property name="imu_slamtec_joint_offset_x" value="0.0"/>
+    <xacro:property name="imu_slamtec_joint_offset_y" value="0.3"/>
     <xacro:property name="imu_slamtec_joint_offset_z" value="${base_height}"/>
 </robot>

Commit message: Flipped back imu positions

File: paxi_ws/src/paxi_description/urdf/include/paxi_imu.xacro (robot description, xacro)
@@ -7,6 +7,6 @@
     <xacro:property name="imu_height" value="0.045"/>
     <!-- should be "inside base box"; -->
-    <xacro:property name="imu_joint_offset_x" value="0.2"/>
-    <xacro:property name="imu_joint_offset_y" value="0.0"/>
+    <xacro:property name="imu_joint_offset_x" value="0.0"/>
+    <xacro:property name="imu_joint_offset_y" value="0.2"/>
     <xacro:property name="imu_joint_offset_z" value="${base_height}"/>
 </robot>

File: paxi_ws/src/paxi_description/urdf/include/paxi_imu_slamtec.xacro (robot description, xacro)
@@ -7,6 +7,6 @@
     <xacro:property name="imu_slamtec_height" value="0.0252"/>
     <!-- should be "inside base box"; -->
-    <xacro:property name="imu_slamtec_joint_offset_x" value="0.0"/>
-    <xacro:property name="imu_slamtec_joint_offset_y" value="0.3"/>
+    <xacro:property name="imu_slamtec_joint_offset_x" value="0.3"/>
+    <xacro:property name="imu_slamtec_joint_offset_y" value="0.0"/>
     <xacro:property name="imu_slamtec_joint_offset_z" value="${base_height}"/>
 </robot>
