Commit message: Updated URDF with new robot build

File: paxi_ws/src/paxi_description/urdf/include/paxi_base.xacro (robot description, xacro)
@@ -3,14 +3,23 @@
     <xacro:property name="baud_rate" value="115200"/>
     <xacro:property name="serial_port" value="/dev/ttyUSB0"/>
-    <xacro:property name="wheel_separation" value="0.42"/>
+    <xacro:property name="wheel_separation" value="0.53"/>
     <xacro:property name="max_velocity" value="100"/>
-    <xacro:property name="base_width" value="0.41"/>
-    <xacro:property name="base_length" value="0.42"/>
-    <xacro:property name="base_height" value="0.01"/>
-    <xacro:property name="base_box_width" value="0.41"/>
-    <xacro:property name="base_box_length" value="0.41"/>
-    <xacro:property name="base_box_height" value="0.21"/>
-    <xacro:property name="base_box_joint_offset_x" value="0.0"/>
+    <xacro:property name="base_width" value="0.46"/>
+    <xacro:property name="base_length" value="0.175"/>
+    <xacro:property name="base_height" value="0.05"/>
+    <xacro:property name="base_box_width" value="0.3302"/>
+    <xacro:property name="base_box_length" value="0.4953"/>
+    <xacro:property name="base_box_height" value="0.2286"/>
+    <xacro:property name="base_box_joint_offset_x" value="0.14"/>
     <xacro:property name="base_box_joint_offset_y" value="0.0"/>
     <xacro:property name="base_box_joint_offset_z" value="${base_height/2 + base_box_height/2}"/>
 </robot>
+ <!--
+ 41.6 - 16.51
+ 43.1 - 16.51
+ y            x           z
+ 19.5 inch * 9 inch * 22 inch box dimensions
+ 49.35 cm  * 33.02 cm box * 55.88cm
+ hoveboard wideth
+ 0.0648
+ -->

File: paxi_ws/src/paxi_description/urdf/include/paxi_imu.xacro (robot description, xacro)
@@ -3,10 +3,10 @@
     <xacro:property name="imu_joint_name" value="imu_joint"/>
     <xacro:property name="imu_link_name" value="imu"/>
-    <xacro:property name="imu_width" value="0.15"/>
-    <xacro:property name="imu_length" value="0.05"/>
-    <xacro:property name="imu_height" value="0.05"/>
+    <xacro:property name="imu_width" value="0.06"/>
+    <xacro:property name="imu_length" value="0.15"/>
+    <xacro:property name="imu_height" value="0.045"/>
     <!-- should be "inside base box"; -->
     <xacro:property name="imu_joint_offset_x" value="0.0"/>
-    <xacro:property name="imu_joint_offset_y" value="0.0"/>
-    <xacro:property name="imu_joint_offset_z" value="${base_height/2 + base_box_height/2}"/>
+    <xacro:property name="imu_joint_offset_y" value="0.20"/>
+    <xacro:property name="imu_joint_offset_z" value="${base_height}"/>
 </robot>

File: paxi_ws/src/paxi_description/urdf/include/paxi_wheels.xacro (robot description, xacro)
@@ -3,9 +3,21 @@
     <xacro:property name="wheel_radius" value="0.086"/>
     <xacro:property name="wheel_length" value="0.05"/>
-    <xacro:property name="wheel_joint_offset_x" value="0.14"/>
+    <!-- <xacro:property name="wheel_joint_offset_x" value="0.14"/>
     <xacro:property name="wheel_joint_offset_y" value="0.255"/>
-    <xacro:property name="caster_wheel_radius" value="0.0375"/>
-    <xacro:property name="caster_wheel_joint_offset_x" value="0.25"/>
+ -->
+    <xacro:property name="wheel_r_joint_offset_x" value="0.0"/>
+    <xacro:property name="wheel_r_joint_offset_y" value="0.2551"/>
+    <xacro:property name="wheel_l_joint_offset_x" value="0.0"/>
+    <xacro:property name="wheel_l_joint_offset_y" value="0.2651"/>
+    <xacro:property name="caster_wheel_radius" value="0.051"/>
+    <xacro:property name="caster_wheel_joint_offset_x" value="0.323"/>
     <xacro:property name="caster_wheel_joint_offset_y" value="0.0"/>
     <xacro:property name="caster_wheel_joint_offset_z" value="0.01"/>
 </robot>
+<!--
+ 41.6 - 16.51
+ 43.1 - 16.51
+ y            x           z
+ 19.5 inch * 13 inch * 22 inch box dimensions
+ 49.35 cm  * 6.5 cm box * 55.88cm
+ -->

File: paxi_ws/src/paxi_description/urdf/paxi_bot.urdf (robot description, URDF)
Before this commit: robot paxi_bot, 9 links, 8 joints
Joints:
- joint ${imu_joint_name}: parent base_box -> base_link
- joint left_wheel_joint: origin xyz=${(-1)*wheel_joint_offset_x} ${wheel_joint_offset_y} 0 rpy=0 0 0 -> xyz=${(-1)*wheel_l_joint_offset_x} ${wheel_l_joint_offset_y} 0 rpy=0 0 0
- joint right_wheel_joint: origin xyz=${(-1)*wheel_joint_offset_x} ${(-1)*wheel_joint_offset_y} 0 rpy=0 0 0 -> xyz=${(-1)*wheel_r_joint_offset_x} ${(-1)*wheel_r_joint_offset_y} 0 rpy=0 0 0

Commit message: Added pitch to robot joints for base box & IMU

File: paxi_ws/src/paxi_description/urdf/include/paxi_base.xacro (robot description, xacro)
@@ -11,4 +11,6 @@
     <xacro:property name="base_box_length" value="0.4953"/>
     <xacro:property name="base_box_height" value="0.2286"/>
+    <!-- tan^-1(2 / 48) -->
+    <xacro:property name ="base_box_angle" value="${math.atan2(2, 48)}"/>
     <xacro:property name="base_box_joint_offset_x" value="0.14"/>
     <xacro:property name="base_box_joint_offset_y" value="0.0"/>

File: paxi_ws/src/paxi_description/urdf/paxi_bot.urdf (robot description, URDF)
Before this commit: robot paxi_bot, 10 links, 9 joints
Joints:
- joint ${imu_joint_name}: origin xyz=${imu_joint_offset_x} ${imu_joint_offset_y} ${imu_joint_offset_z} rpy=0 0 0 -> xyz=${imu_joint_offset_x} ${imu_joint_offset_y} ${imu_joint_offset_z} rpy=0 ${base_box_angle} 0
- joint ${imu_slamtec_joint_name}: origin xyz=${imu_slamtec_joint_offset_x} ${imu_slamtec_joint_offset_y} ${imu_slamtec_joint_offset_z} rpy=0 0 0 -> xyz=${imu_slamtec_joint_offset_x} ${imu_slamtec_joint_offset_y} ${imu_slamtec_joint_offset_z} rpy=0 ${base_box_angle} 0
- joint base_box_joint: origin xyz=${base_box_joint_offset_x} ${base_box_joint_offset_y} ${base_box_joint_offset_z} rpy=0 0 0 -> xyz=${base_box_joint_offset_x} ${base_box_joint_offset_y} ${base_box_joint_offset_z} rpy=0 ${base_box_angle} 0

Commit message: Updated default usb device names with better reproducible names via udevadm symlink

File: paxi_ws/src/paxi_description/urdf/include/paxi_base.xacro (robot description, xacro)
@@ -2,5 +2,5 @@
 <robot name="paxi_bot" xmlns:xacro="http://www.ros.org/wiki/xacro">
     <xacro:property name="baud_rate" value="115200"/>
-    <xacro:property name="serial_port" value="/dev/ttyUSB0"/>
+    <xacro:property name="serial_port" value="/dev/hoverboard_serial"/>
     <xacro:property name="wheel_separation" value="0.53"/>
     <xacro:property name="max_velocity" value="100"/>
