Commit message: update wheel radius to 0.084

File: paxi_ws/src/paxi_description/urdf/include/paxi_wheels.xacro (robot description, xacro)
@@ -1,5 +1,7 @@
 <?xml version="1.0"?>
 <robot name="paxi_bot" xmlns:xacro="http://www.ros.org/wiki/xacro">
-    <xacro:property name="wheel_radius" value="0.086"/>
+<!-- closest thing i found to a data sheet for these wheels specifically:  -->
+<!-- https://www.parallax.com/product/6-5-hub-motor-with-encoder/ -->
+    <xacro:property name="wheel_radius" value="0.084"/>
     <xacro:property name="wheel_length" value="0.05"/>
     <!-- <xacro:property name="wheel_joint_offset_x" value="0.14"/>
