Commit message: rviz launch for nav2 added, setting up ekf

File: paxi_ws/src/paxi_description/urdf/paxi_bot.urdf (robot description, URDF)
Before this commit: robot paxi_bot, 7 links, 6 joints
Joints:
- joint caster_wheel_joint: origin xyz=${caster_wheel_joint_offset_x} ${caster_wheel_joint_offset_y} ${caster_wheel_joint_offset_z} rpy=0 0 0 -> xyz=${caster_wheel_joint_offset_x} ${caster_wheel_joint_offset_y} ${-1*caster_wheel_joint_offset_z} rpy=0 0 0

Commit message: URDF fixed left wheel direction

File: paxi_ws/src/paxi_description/urdf/paxi_bot.urdf (robot description, URDF)
Before this commit: robot paxi_bot, 7 links, 6 joints
Joints:
- joint left_wheel_joint: axis 0 1 0 -> 0 -1 0

Commit message: Build and live test, fixed flipped orientation in wheel postition/velocity data

File: paxi_ws/src/paxi_description/urdf/paxi_bot.urdf (robot description, URDF)
Before this commit: robot paxi_bot, 7 links, 6 joints
Joints:
- joint left_wheel_joint: axis 0 -1 0 -> 0 1 0

Commit message: added box to urdf, still need to fix its offset

File: paxi_ws/src/paxi_description/urdf/paxi_bot.urdf (robot description, URDF)
Before this commit: robot paxi_bot, 7 links, 6 joints
Links:
- added link base_box; visual box size=${base_box_length} ${base_box_width} ${base_box_height}
Joints:
- added joint base_box_joint: type fixed, parent base_link, child base_box, origin xyz=${base_box_joint_offset_x} ${base_box_joint_offset_y} ${base_box_joint_offset_z} rpy=0 0 0

Commit message: Fixed URDF and added lidar box

File: paxi_ws/src/paxi_description/urdf/paxi_bot.urdf (robot description, URDF)
Before this commit: robot paxi_bot, 8 links, 7 joints
Links:
- removed link imu_link
- added link lidar_box; visual box size=${lidar_box_length} ${lidar_box_width} ${lidar_box_height}
Joints:
- removed joint imu_joint
- added joint lidar_box_joint: type fixed, parent base_box, child lidar_box, origin xyz=${lidar_box_joint_offset_x} ${lidar_box_joint_offset_y} ${lidar_box_joint_offset_z} rpy=0 0 0
- joint base_scan_joint: parent base_link -> lidar_box

Commit message: Fixed and Cleaned URDF again

File: paxi_ws/src/paxi_description/urdf/paxi_bot.urdf (robot description, URDF)
Before this commit: robot paxi_bot, 8 links, 7 joints
Joints:
- joint base_scan_joint: origin xyz=${lidar_joint_offset_x} ${lidar_joint_offset_y} ${lidar_joint_offset_z} rpy=0 0 0 -> xyz=0 0 ${lidar_joint_offset_z} rpy=0 0 0
- joint caster_wheel_joint: origin xyz=${caster_wheel_joint_offset_x} ${caster_wheel_joint_offset_y} ${-1*caster_wheel_joint_offset_z} rpy=0 0 0 -> xyz=${caster_wheel_joint_offset_x} ${caster_wheel_joint_offset_y} ${caster_wheel_joint_offset_z} rpy=0 0 0

Commit message: Updated urdf to have imu, and link/joint name as XACRO parameter

File: paxi_ws/src/paxi_description/urdf/paxi_bot.urdf (robot description, URDF)
Before this commit: robot paxi_bot, 8 links, 7 joints
Links:
- added link {$imu_link_name}; visual box size=${imu_length} ${lidar_box_width} ${lidar_box_height}
Joints:
- added joint ${imu_joint_name}: type fixed, parent base_box, child ${imu_link_name}, origin xyz=${imu_joint_offset_x} ${lidar_box_joint_offset_y} ${lidar_box_joint_offset_z} rpy=0 0 0

Commit message: EKF IMU smoothed out, Controller yaml updated base_link set to base footprint

File: paxi_ws/src/paxi_description/urdf/paxi_bot.urdf (robot description, URDF)
Before this commit: robot paxi_bot, 9 links, 8 joints
Joints:
- joint base_scan_joint: origin xyz=0 0 ${lidar_joint_offset_z} rpy=0 0 0 -> xyz=0 0 ${lidar_joint_offset_z} rpy=0 0 ${pi}

Commit message: Added roatation of pi (180 degrees) in imu_slamtex urdf

File: paxi_ws/src/paxi_description/urdf/paxi_bot.urdf (robot description, URDF)
Before this commit: robot paxi_bot, 10 links, 9 joints
Joints:
- joint ${imu_joint_name}: origin xyz=${imu_joint_offset_x} ${imu_joint_offset_y} ${imu_joint_offset_z} rpy=0 ${base_box_angle} 0 -> xyz=${imu_joint_offset_x} ${imu_joint_offset_y} ${imu_joint_offset_z} rpy=0 ${base_box_angle} ${pi}

Commit message: pi rotation placed on wrong joint

File: paxi_ws/src/paxi_description/urdf/paxi_bot.urdf (robot description, URDF)
Before this commit: robot paxi_bot, 10 links, 9 joints
Joints:
- joint ${imu_joint_name}: origin xyz=${imu_joint_offset_x} ${imu_joint_offset_y} ${imu_joint_offset_z} rpy=0 ${base_box_angle} ${pi} -> xyz=${imu_joint_offset_x} ${imu_joint_offset_y} ${imu_joint_offset_z} rpy=0 ${base_box_angle} 0
- joint ${imu_slamtec_joint_name}: origin xyz=${imu_slamtec_joint_offset_x} ${imu_slamtec_joint_offset_y} ${imu_slamtec_joint_offset_z} rpy=0 ${base_box_angle} 0 -> xyz=${imu_slamtec_joint_offset_x} ${imu_slamtec_joint_offset_y} ${imu_slamtec_joint_offset_z} rpy=0 ${base_box_angle} {pi}

Commit message: fixed "${pi}" to correctly get xacro param"

File: paxi_ws/src/paxi_description/urdf/paxi_bot.urdf (robot description, URDF)
Before this commit: robot paxi_bot, 10 links, 9 joints
Joints:
- joint ${imu_slamtec_joint_name}: origin xyz=${imu_slamtec_joint_offset_x} ${imu_slamtec_joint_offset_y} ${imu_slamtec_joint_offset_z} rpy=0 ${base_box_angle} {pi} -> xyz=${imu_slamtec_joint_offset_x} ${imu_slamtec_joint_offset_y} ${imu_slamtec_joint_offset_z} rpy=0 ${base_box_angle} ${pi}

Commit message: Removed ${pi} rotation imu frames, correct rpy added to imu_hover and imu_slamtec

File: paxi_ws/src/paxi_description/urdf/paxi_bot.urdf (robot description, URDF)
Before this commit: robot paxi_bot, 10 links, 9 joints
Joints:
- joint ${imu_slamtec_joint_name}: origin xyz=${imu_slamtec_joint_offset_x} ${imu_slamtec_joint_offset_y} ${imu_slamtec_joint_offset_z} rpy=0 ${base_box_angle} ${pi} -> xyz=${imu_slamtec_joint_offset_x} ${imu_slamtec_joint_offset_y} ${imu_slamtec_joint_offset_z} rpy=0 ${base_box_angle} 0

Commit message: IMU links now with correct orientation viaully and on joint

File: paxi_ws/src/paxi_description/urdf/paxi_bot.urdf (robot description, URDF)
Before this commit: robot paxi_bot, 10 links, 9 joints
Joints:
- joint ${imu_joint_name}: origin xyz=${imu_joint_offset_x} ${imu_joint_offset_y} ${imu_joint_offset_z} rpy=0 ${base_box_angle} 0 -> xyz=${imu_joint_offset_x} ${imu_joint_offset_y} ${imu_joint_offset_z} rpy=0 0 0
