Commit message: Simulation Port complete, need to add mass/inertia to all link and joints. but robot spwans in gz-sim and responds to teleop twist (but not correctly)

File: paxi_ws/src/paxi_description/urdf/paxi_bot_simulation.urdf (robot description, URDF)
Before this commit: robot paxi_bot, 10 links, 9 joints
Links:
- link base_footprint: mass None -> 0.0001
- link base_link: mass None -> 10.0
- link caster_wheel: mass None -> 0.5; geometry collision sphere radius=${caster_wheel_radius}; visual sphere radius=${caster_wheel_radius}
- link left_wheel: mass None -> 5.0; geometry collision cylinder length=${wheel_length} radius=${wheel_radius}; visual cylinder length=${wheel_length} radius=${wheel_radius}
- link right_wheel: mass None -> 5.0; geometry collision cylinder length=${wheel_length} radius=${wheel_radius}; visual cylinder length=${wheel_length} radius=${wheel_radius}

Commit message: ADded ineertials, fixed incorrect urdf

File: paxi_ws/src/paxi_description/urdf/paxi_bot_simulation.urdf (robot description, URDF)
Before this commit: robot paxi_bot, 10 links, 9 joints
Links:
- link base_link: mass 10.0 -> None
- link caster_wheel: mass 0.5 -> None
- link left_wheel: mass 5.0 -> None
- link right_wheel: mass 5.0 -> None

File: paxi_ws/src/paxi_description/urdf/simulation/paxi_base_inertials.xacro (robot description, xacro)
@@ -1,38 +1,38 @@
 <?xml version="1.0"?>
 <robot name="paxi_bot" xmlns:xacro="http://www.ros.org/wiki/xacro">
-     <xacro:property name = "base_link_ixx" value = 0.0>
-     <xacro:property name = "base_link_ixy" value = 0.0>
-     <xacro:property name = "base_link_ixz" value = 0.0>
-     <xacro:property name = "base_link_iyx" value = 0.0>
-     <xacro:property name = "base_link_iyy" value = 0.0>
-     <xacro:property name = "base_link_iyz" value = 0.0>
-     <xacro:property name = "base_link_izx" value = 0.0>
-     <xacro:property name = "base_link_izy" value = 0.0>
-     <xacro:property name = "base_link_izz" value = 0.0>
-     <xacro:property name = "base_link_mass" value = 6.5kg>
+     <xacro:property name = "base_link_ixx" value = "0.01784167"/>
+     <xacro:property name = "base_link_ixy" value = "0.0"/>
+     <xacro:property name = "base_link_ixz" value = "0.0"/>
+     <xacro:property name = "base_link_iyx" value = "0.0"/>
+     <xacro:property name = "base_link_iyy" value = "0.00276042"/>
+     <xacro:property name = "base_link_iyz" value = "0.0"/>
+     <xacro:property name = "base_link_izx" value = "0.0"/>
+     <xacro:property name = "base_link_izy" value = "0.0"/>
+     <xacro:property name = "base_link_izz" value = "0.02018542"/>
+     <xacro:property name = "base_link_mass" value = "6.5"/>
      <xacro:macro name="base_link_inertial">
           <inertial>
-               <mass value="$base_link_mass" />
-               <inertia  ixx="$base_link_mass*{base_link_ixx}"   iyz="$base_link_mass*{base_link_ixy}"  izx="$base_link_mass*{base_link_izx}"
-                         ixy="$base_link_mass*{base_link_iyy}"   iyy="$base_link_mass*{base_link_iyy}"  izy="$base_link_mass*{base_link_izy}"
-                         ixz="$base_link_mass*{base_link_iyy}"   iyz="$base_link_mass*{base_link_iyz}"  izz="$base_link_mass*{base_link_izz}"  />
+               <mass value="${base_link_mass}" />
+               <inertia  ixx="${base_link_mass*base_link_ixx}"   ixy="${base_link_mass*base_link_ixy}"  ixz="${base_link_mass*base_link_ixz}"
+                         iyx="${base_link_mass*base_link_iyx}"   iyy="${base_link_mass*base_link_iyy}"  iyz="${base_link_mass*base_link_iyz}"
+                         izx="${base_link_mass*base_link_izx}"   izy="${base_link_mass*base_link_izy}"  izz="${base_link_mass*base_link_izz}"/>
           </inertial>
      </xacro:macro>
-     <xacro:property name = "base_box_ixx" value = 0.0>
-     <xacro:property name = "base_box_ixy" value = 0.0>
-     <xacro:property name = "base_box_ixz" value = 0.0>
-     <xacro:property name = "base_box_iyx" value = 0.0>
-     <xacro:property name = "base_box_iyy" value = 0.0>
-     <xacro:property name = "base_box_iyz" value = 0.0>
-     <xacro:property name = "base_box_izx" value = 0.0>
-     <xacro:property name = "base_box_izy" value = 0.0>
-     <xacro:property name = "base_box_izz" value = 0.0>
-     <xacro:property name = "base_box_mass" value = ${3.5 + 1.58 + 1.77 + 0.05}>
+     <xacro:property name = "base_box_ixx" value = "0.013440833333333332"/>
+     <xacro:property name = "base_box_ixy" value = "0.0"/>
+     <xacro:property name = "base_box_ixz" value = "0.0"/>
+     <xacro:property name = "base_box_iyx" value = "0.0"/>
+     <xacro:property name = "base_box_iyy" value = "0.024798337500000003"/>
+     <xacro:property name = "base_box_iyz" value = "0.0"/>
+     <xacro:property name = "base_box_izx" value = "0.0"/>
+     <xacro:property name = "base_box_izy" value = "0.0"/>
+     <xacro:property name = "base_box_izz" value = "0.029529510833333335"/>
+     <xacro:property name = "base_box_mass" value = "${3.5 + 1.58 + 1.77 + 0.05}"/>
      <xacro:macro name="base_box_inertial">
           <inertial>
-               <mass value="${base_box_mass}" />
-               <inertia  ixx="$base_box_mass*{base_box_ixx}"   iyz="$base_box_mass*{base_box_ixy}"  izx="$base_box_mass*{base_box_izx}"
-                         ixy="$base_box_mass*{base_box_iyy}"   iyy="$base_box_mass*{base_box_iyy}"  izy="$base_box_mass*{base_box_izy}"
-                         ixz="$base_box_mass*{base_box_iyy}"   iyz="$base_box_mass*{base_box_iyz}"  izz="$base_box_mass*{base_box_izz}"  />
+               <mass value="${base_box_mass}"/>
+               <inertia  ixx="${base_box_mass*base_box_ixx}"   ixy="${base_box_mass*base_box_ixy}"  ixz="${base_box_mass*base_box_ixz}"
+                         iyx="${base_box_mass*base_box_iyx}"   iyy="${base_box_mass*base_box_iyy}"  iyz="${base_box_mass*base_box_iyz}"
+                         izx="${base_box_mass*base_box_izx}"   izy="${base_box_mass*base_box_izx}"  izz="${base_box_mass*base_box_izz}"  />
           </inertial>
      </xacro:macro>

File: paxi_ws/src/paxi_description/urdf/simulation/paxi_imu_inertials.xacro (robot description, xacro)
@@ -1,20 +1,20 @@
 <?xml version="1.0"?>
 <robot name="paxi_bot" xmlns:xacro="http://www.ros.org/wiki/xacro">
-     <xacro:property name = "imu_hover_ixx" value = 0.0>
-     <xacro:property name = "imu_hover_ixy" value = 0.0>
-     <xacro:property name = "imu_hover_ixz" value = 0.0>
-     <xacro:property name = "imu_hover_iyx" value = 0.0>
-     <xacro:property name = "imu_hover_iyy" value = 0.0>
-     <xacro:property name = "imu_hover_iyz" value = 0.0>
-     <xacro:property name = "imu_hover_izx" value = 0.0>
-     <xacro:property name = "imu_hover_izy" value = 0.0>
-     <xacro:property name = "imu_hover_izz" value = 0.0>
-     <xacro:property name = "imu_hover_mass" value = 0.01>
+     <xacro:property name = "imu_hover_ixx" value = "0.00046875"/>
+     <xacro:property name = "imu_hover_ixy" value = "0.0"/>
+     <xacro:property name = "imu_hover_ixz" value = "0.0"/>
+     <xacro:property name = "imu_hover_iyx" value = "0.0"/>
+     <xacro:property name = "imu_hover_iyy" value = "0.0020437499999999996"/>
+     <xacro:property name = "imu_hover_iyz" value = "0.0"/>
+     <xacro:property name = "imu_hover_izx" value = "0.0"/>
+     <xacro:property name = "imu_hover_izy" value = "0.0"/>
+     <xacro:property name = "imu_hover_izz" value = "0.002175"/>
+     <xacro:property name = "imu_hover_mass" value = "0.0001"/>
      <xacro:macro name="imu_hover_inertial">
         <inertial>
-            <mass value="${imu_hover_mass}" />
-            <inertia    ixx="${imu_mass}{imu_hover_ixx}"   iyz="${imu_mass}{imu_hover_ixy}"  izx="${imu_mass}{imu_hover_izx}"
-                        ixy="${imu_mass}{imu_hover_iyy}"   iyy="${imu_mass}{imu_hover_iyy}"  izy="${imu_mass}{imu_hover_izy}"
-                        ixz="${imu_mass}{imu_hover_iyy}"   iyz="${imu_mass}{imu_hover_iyz}"  izz="${imu_mass}{imu_hover_izz}"  />
+            <mass value="${imu_hover_mass}"/>
+            <inertia    ixx="${imu_hover_mass*imu_hover_ixx}"  ixy="${imu_hover_mass*imu_hover_ixy}"  ixz="${imu_hover_mass*imu_hover_ixz}"
+                        iyx="${imu_hover_mass*imu_hover_iyx}"  iyy="${imu_hover_mass*imu_hover_iyy}"  iyz="${imu_hover_mass*imu_hover_iyz}"
+                        izx="${imu_hover_mass*imu_hover_izx}"  izy="${imu_hover_mass*imu_hover_izy}"  izz="${imu_hover_mass*imu_hover_izz}" />
         </inertial>
      </xacro:macro>

File: paxi_ws/src/paxi_description/urdf/simulation/paxi_imu_slamtec_inertials.xacro (robot description, xacro)
@@ -1,20 +1,20 @@
 <?xml version="1.0"?>
 <robot name="paxi_bot" xmlns:xacro="http://www.ros.org/wiki/xacro">
-     <xacro:property name = "imu_ixx" value = 0.0>
-     <xacro:property name = "imu_ixy" value = 0.0>
-     <xacro:property name = "imu_ixz" value = 0.0>
-     <xacro:property name = "imu_iyx" value = 0.0>
-     <xacro:property name = "imu_iyy" value = 0.0>
-     <xacro:property name = "imu_iyz" value = 0.0>
-     <xacro:property name = "imu_izx" value = 0.0>
-     <xacro:property name = "imu_izy" value = 0.0>
-     <xacro:property name = "imu_izz" value = 0.0>
-     <xacro:property name = "imu_mass" value = 0.01>
-     <xacro:macro name="imu_inertial">
+     <xacro:property name = "imu_ixx" value = "0.0002513733333333333"/>
+     <xacro:property name = "imu_ixy" value = "0.0"/>
+     <xacro:property name = "imu_ixz" value = "0.0"/>
+     <xacro:property name = "imu_iyx" value = "0.0"/>
+     <xacro:property name = "imu_iyy" value = "0.0002941233333333333"/>
+     <xacro:property name = "imu_iyz" value = "0.0"/>
+     <xacro:property name = "imu_izx" value = "0.0"/>
+     <xacro:property name = "imu_izy" value = "0.0"/>
+     <xacro:property name = "imu_izz" value = "0.00043965666666666666"/>
+     <xacro:property name = "imu_mass" value = "0.01"/>
+     <xacro:macro name="imu_slamtec_inertial">
         <inertial>
             <mass value="${imu_mass}" />
-            <inertia    ixx="${imu_mass}*{imu_ixx}"   iyz="${imu_mass}*{imu_ixy}"  izx="${imu_mass}*{imu_izx}"
-                        ixy="${imu_mass}*{imu_iyy}"   iyy="${imu_mass}*{imu_iyy}"  izy="${imu_mass}*{imu_izy}"
-                        ixz="${imu_mass}*{imu_iyy}"   iyz="${imu_mass}*{imu_iyz}"  izz="${imu_mass}*{imu_izz}"  />
+            <inertia    ixx="${imu_mass*imu_ixx}"   ixy="${imu_mass*imu_ixy}"  ixz="${imu_mass*imu_ixz}"
+                        iyx="${imu_mass*imu_iyx}"   iyy="${imu_mass*imu_iyy}"  iyz="${imu_mass*imu_iyz}"
+                        izx="${imu_mass*imu_izx}"   izy="${imu_mass*imu_izy}"  izz="${imu_mass*imu_izz}"  />
         </inertial>
      </xacro:macro>

File: paxi_ws/src/paxi_description/urdf/simulation/paxi_lidar_inertials.xacro (robot description, xacro)
@@ -1,40 +1,40 @@
 <?xml version="1.0"?>
 <robot name="paxi_bot" xmlns:xacro="http://www.ros.org/wiki/xacro">
-    <xacro:property name = "lidar_ixx" value = 0.0>
-    <xacro:property name = "lidar_ixy" value = 0.0>
-    <xacro:property name = "lidar_ixz" value = 0.0>
-    <xacro:property name = "lidar_iyx" value = 0.0>
-    <xacro:property name = "lidar_iyy" value = 0.0>
-    <xacro:property name = "lidar_iyz" value = 0.0>
-    <xacro:property name = "lidar_izx" value = 0.0>
-    <xacro:property name = "lidar_izy" value = 0.0>
-    <xacro:property name = "lidar_izz" value = 0.0>
+    <xacro:property name = "lidar_ixx" value = "0.00028958333333333337"/>
+    <xacro:property name = "lidar_ixy" value = "0.0"/>
+    <xacro:property name = "lidar_ixz" value = "0.0"/>
+    <xacro:property name = "lidar_iyx" value = "0.0"/>
+    <xacro:property name = "lidar_iyy" value = "0.00028958333333333337"/>
+    <xacro:property name = "lidar_iyz" value = "0.0"/>
+    <xacro:property name = "lidar_izx" value = "0.0"/>
+    <xacro:property name = "lidar_izy" value = "0.0"/>
+    <xacro:property name = "lidar_izz" value = "0.0031250000000000006"/>
     <!-- https://bucket-download.slamtec.com/9fd56b14eb46b11ffb38d861db4a7771c70e3095/SLAMTEC_rplidar_datasheet_C1_v1.2_en.pdf -->
-    <xacro:property name = "mass" value = 0.110 >
+    <xacro:property name = "lidar_mass" value = "0.110" />
     <xacro:macro name="lidar_inertial">
         <inertial>
-            <mass value="${lidar_mass}" />
-            <inertia    ixx="${mass}*{lidar_ixx}"   iyz="${mass}*{lidar_ixy}"  izx="${mass}*{lidar_izx}"
-                        ixy="${mass}*{lidar_iyy}"   iyy="${mass}*{lidar_iyy}"  izy="${mass}*{lidar_izy}"
-                        ixz="${mass}*{lidar_iyy}"   iyz="${mass}*{lidar_iyz}"  izz="${mass}*{lidar_izz}"  />
+            <mass value="${lidar_mass}"/>
+            <inertia ixx="${lidar_mass*lidar_ixx}"  ixy="${lidar_mass*lidar_ixy}"  ixz="${lidar_mass*lidar_ixz}"
+                    iyx="${lidar_mass*lidar_iyx}"  iyy="${lidar_mass*lidar_iyy}"  iyz="${lidar_mass*lidar_iyz}"
+                    izx="${lidar_mass*lidar_izx}"  izy="${lidar_mass*lidar_izy}"  izz="${lidar_mass*lidar_izz}"/>
         </inertial>
     </xacro:macro>
-    <xacro:property name = "lidar_box_ixx" value = 0.0>
-    <xacro:property name = "lidar_box_ixy" value = 0.0>
-    <xacro:property name = "lidar_box_ixz" value = 0.0>
-    <xacro:property name = "lidar_box_iyx" value = 0.0>
-    <xacro:property name = "lidar_box_iyy" value = 0.0>
-    <xacro:property name = "lidar_box_iyz" value = 0.0>
-    <xacro:property name = "lidar_box_izx" value = 0.0>
-    <xacro:property name = "lidar_box_izy" value = 0.0>
-    <xacro:property name = "lidar_box_izz" value = 0.0>
-    <xacro:property name = "lidar_box_inertial" value = 0.01>
+    <xacro:property name = "lidar_box_ixx" value = "0.0007416666666666667"/>
+    <xacro:property name = "lidar_box_ixy" value = "0.0"/>
+    <xacro:property name = "lidar_box_ixz" value = "0.0"/>
+    <xacro:property name = "lidar_box_iyx" value = "0.0"/>
+    <xacro:property name = "lidar_box_iyy" value = "0.01408333333333333"/>
+    <xacro:property name = "lidar_box_iyz" value = "0.0"/>
+    <xacro:property name = "lidar_box_izx" value = "0.0"/>
+    <xacro:property name = "lidar_box_izy" value = "0.0"/>
+    <xacro:property name = "lidar_box_izz" value = "0.0017333333333333333"/>
+    <xacro:property name = "lidar_box_mass" value = "0.01"/>
     <xacro:macro name="lidar_box_inertial">
         <inertial>
             <mass value="${lidar_box_mass}" />
-            <inertia    ixx="${mass}*{lidar_ixx}"   iyz="${mass}*{lidar_ixy}"  izx="${mass}*{lidar_izx}"
-                        ixy="${mass}*{lidar_iyy}"   iyy="${mass}*{lidar_iyy}"  izy="${mass}*{lidar_izy}"
-                        ixz="${mass}*{lidar_iyy}"   iyz="${mass}*{lidar_iyz}"  izz="${mass}*{lidar_izz}"  />
-        </inertial>
+            <inertia ixx="${lidar_box_mass*lidar_box_ixx}"  ixy="${lidar_box_mass*lidar_box_ixy}"  ixz="${lidar_box_mass*lidar_box_ixz}"
+                    iyx="${lidar_box_mass*lidar_box_iyx}"  iyy="${lidar_box_mass*lidar_box_iyy}"  iyz="${lidar_box_mass*lidar_box_iyz}"
+                    izx="${lidar_box_mass*lidar_box_izx}"  izy="${lidar_box_mass*lidar_box_izy}"  izz="${lidar_box_mass*lidar_box_izz}"/>
+            </inertial>
     </xacro:macro>
 </robot>

File: paxi_ws/src/paxi_description/urdf/simulation/paxi_wheels_inertials.xacro (robot description, xacro)
@@ -1,58 +1,58 @@
 <?xml version="1.0"?>
 <robot name="paxi_bot" xmlns:xacro="http://www.ros.org/wiki/xacro">
-    <xacro:property name = "left_wheel_ixx" value = 0.0>
-    <xacro:property name = "left_wheel_ixy" value = 0.0>
-    <xacro:property name = "left_wheel_ixz" value = 0.0>
-    <xacro:property name = "left_wheel_iyx" value = 0.0>
-    <xacro:property name = "left_wheel_iyy" value = 0.0>
-    <xacro:property name = "left_wheel_iyz" value = 0.0>
-    <xacro:property name = "left_wheel_izx" value = 0.0>
-    <xacro:property name = "left_wheel_izy" value = 0.0>
-    <xacro:property name = "left_wheel_izz" value = 0.0>
+    <xacro:property name = "left_wheel_ixx" value = "0.0028958333333333337"/>
+    <xacro:property name = "left_wheel_ixy" value = "0.0"/>
+    <xacro:property name = "left_wheel_ixz" value = "0.0"/>
+    <xacro:property name = "left_wheel_iyx" value = "0.0"/>
+    <xacro:property name = "left_wheel_iyy" value = "0.002057333333333333"/>
+    <xacro:property name = "left_wheel_iyz" value = "0.0"/>
+    <xacro:property name = "left_wheel_izx" value = "0.0"/>
+    <xacro:property name = "left_wheel_izy" value = "0.0"/>
+    <xacro:property name = "left_wheel_izz" value = "0.0036979999999999995"/>
     <!-- ref: https://www.parallax.com/product/6-5-hub-motor-with-encoder/ -->
-    <xacro:property name = "left_wheel_mass" value = 3.1>
+    <xacro:property name = "left_wheel_mass" value = "3.1"/>
     <xacro:macro name="left_wheel_inertial">
         <inertial>
-            <mass value="${mass}" />
-            <inertia    ixx="${left_wheel_mass}*{left_wheel_ixx}"   iyz="${left_wheel_mass}*{left_wheel_ixy}"  izx="${left_wheel_mass}*{left_wheel_izx}"
-                        ixy="${left_wheel_mass}*{left_wheel_iyy}"   iyy="${left_wheel_mass}*{left_wheel_iyy}"  izy="${left_wheel_mass}*{left_wheel_izy}"
-                        ixz="${left_wheel_mass}*{left_wheel_iyy}"   iyz="${left_wheel_mass}*{left_wheel_iyz}"  izz="${left_wheel_mass}*{left_wheel_izz}"  />
+            <mass value="${left_wheel_mass}" />
+            <inertia    ixx="${left_wheel_mass*left_wheel_ixx}"   ixy="${left_wheel_mass*left_wheel_ixy}"  ixz="${left_wheel_mass*left_wheel_ixz}"
+                        iyx="${left_wheel_mass*left_wheel_iyx}"   iyy="${left_wheel_mass*left_wheel_iyy}"  iyz="${left_wheel_mass*left_wheel_iyz}"
+                        izx="${left_wheel_mass*left_wheel_izx}"   izy="${left_wheel_mass*left_wheel_izy}"  izz="${left_wheel_mass*left_wheel_izz}"  />
         </inertial>
     </xacro:macro>
-    <xacro:property name = "right_wheel_ixx" value = 0.0>
-    <xacro:property name = "right_wheel_ixy" value = 0.0>
-    <xacro:property name = "right_wheel_ixz" value = 0.0>
-    <xacro:property name = "right_wheel_iyx" value = 0.0>
-    <xacro:property name = "right_wheel_iyy" value = 0.0>
-    <xacro:property name = "right_wheel_iyz" value = 0.0>
-    <xacro:property name = "right_wheel_izx" value = 0.0>
-    <xacro:property name = "right_wheel_izy" value = 0.0>
-    <xacro:property name = "right_wheel_izz" value = 0.0>
+    <xacro:property name = "right_wheel_ixx" value = "0.0028958333333333337"/>
+    <xacro:property name = "right_wheel_ixy" value = "0.0"/>
+    <xacro:property name = "right_wheel_ixz" value = "0.0"/>
+    <xacro:property name = "right_wheel_iyx" value = "0.0"/>
+    <xacro:property name = "right_wheel_iyy" value = "0.002057333333333333"/>
+    <xacro:property name = "right_wheel_iyz" value = "0.0"/>
+    <xacro:property name = "right_wheel_izx" value = "0.0"/>
+    <xacro:property name = "right_wheel_izy" value = "0.0"/>
+    <xacro:property name = "right_wheel_izz" value = "0.0036979999999999995"/>
     <!-- ref: https://www.parallax.com/product/6-5-hub-motor-with-encoder/ -->
-    <xacro:property name = "right_wheel_mass" value = 3.1>
+    <xacro:property name = "right_wheel_mass" value = "3.1"/>
     <xacro:macro name="right_wheel_inertial">
         <inertial>
-            <mass value="${mass}" />
-            <inertia    ixx="${right_wheel_mass}*{right_wheel_ixx}"   iyz="${right_wheel_mass}*{right_wheel_ixy}"  izx="${right_wheel_mass}*{right_wheel_izx}"
-                        ixy="${right_wheel_mass}*{right_wheel_iyy}"   iyy="${right_wheel_mass}*{right_wheel_iyy}"  izy="${right_wheel_mass}*{right_wheel_izy}"
-                        ixz="${right_wheel_mass}*{right_wheel_iyy}"   iyz="${right_wheel_mass}*{right_wheel_iyz}"  izz="${right_wheel_mass}*{right_wheel_izz}"  />
+            <mass value="${right_wheel_mass}" />
+            <inertia    ixx="${right_wheel_mass*right_wheel_ixx}"   ixy="${right_wheel_mass*right_wheel_ixy}"  ixz="${right_wheel_mass*right_wheel_ixz}"
+                        iyx="${right_wheel_mass*right_wheel_iyx}"   iyy="${right_wheel_mass*right_wheel_iyy}"  iyz="${right_wheel_mass*right_wheel_iyz}"
+                        izx="${right_wheel_mass*right_wheel_izx}"   izy="${right_wheel_mass*right_wheel_izy}"  izz="${right_wheel_mass*right_wheel_izz}"  />
         </inertial>
     </xacro:macro>
-    <xacro:property name = "caster_wheel_ixx" value = 0.0>
-    <xacro:property name = "caster_wheel_ixy" value = 0.0>
-    <xacro:property name = "caster_wheel_ixz" value = 0.0>
-    <xacro:property name = "caster_wheel_iyx" value = 0.0>
-    <xacro:property name = "caster_wheel_iyy" value = 0.0>
-    <xacro:property name = "caster_wheel_iyz" value = 0.0>
-    <xacro:property name = "caster_wheel_izx" value = 0.0>
-    <xacro:property name = "caster_wheel_izy" value = 0.0>
-    <xacro:property name = "caster_wheel_izz" value = 0.0>
-    <xacro:property name = "caster_wheel_mass" value = 0.110>
+    <xacro:property name = "caster_wheel_ixx" value = "0.0010404"/>
+    <xacro:property name = "caster_wheel_ixy" value = "0.0"/>
+    <xacro:property name = "caster_wheel_ixz" value = "0.0"/>
+    <xacro:property name = "caster_wheel_iyx" value = "0.0"/>
+    <xacro:property name = "caster_wheel_iyy" value = "0.0010404"/>
+    <xacro:property name = "caster_wheel_iyz" value = "0.0"/>
+    <xacro:property name = "caster_wheel_izx" value = "0.0"/>
+    <xacro:property name = "caster_wheel_izy" value = "0.0"/>
+    <xacro:property name = "caster_wheel_izz" value = "0.0010404"/>
+    <xacro:property name = "caster_wheel_mass" value = "0.110"/>
     <xacro:macro name="caster_wheel_inertial">
          <inertial>
-            <mass value="${caster_mass}" />
-            <inertia    ixx="${caster_mass}*{caster_wheel_ixx}"   iyz="${caster_mass}*{caster_wheel_ixy}"  izx="${caster_mass}*{caster_wheel_izx}"
-                        ixy="${caster_mass}*{caster_wheel_iyy}"   iyy="${caster_mass}*{caster_wheel_iyy}"  izy="${caster_mass}*{caster_wheel_izy}"
-                        ixz="${caster_mass}*{caster_wheel_iyy}"   iyz="${caster_mass}*{caster_wheel_iyz}"  izz="${caster_mass}*{caster_wheel_izz}"  />
+            <mass value="${caster_wheel_mass}" />
+            <inertia    ixx="${caster_wheel_mass*caster_wheel_ixx}"   ixy="${caster_wheel_mass*caster_wheel_ixy}"  ixz="${caster_wheel_mass*caster_wheel_ixz}"
+                        iyx="${caster_wheel_mass*caster_wheel_iyx}"   iyy="${caster_wheel_mass*caster_wheel_iyy}"  iyz="${caster_wheel_mass*caster_wheel_iyz}"
+                        izx="${caster_wheel_mass*caster_wheel_izx}"   izy="${caster_wheel_mass*caster_wheel_izy}"  izz="${caster_wheel_mass*caster_wheel_izz}"  />
         </inertial>
     </xacro:macro>
