Commit message: update inertial values in simulation

File: paxi_ws/src/paxi_description/urdf/paxi_bot_simulation.urdf (robot description, URDF)
Before this commit: robot paxi_bot, 10 links, 9 joints
Links:
- link base_footprint: mass 0.0001 -> None

File: paxi_ws/src/paxi_description/urdf/simulation/paxi_base_inertials.xacro (robot description, xacro)
@@ -1,20 +1,23 @@
 <?xml version="1.0"?>
 <robot name="paxi_bot" xmlns:xacro="http://www.ros.org/wiki/xacro">
-     <xacro:property name = "base_link_ixx" value = "0.01784167"/>
+     <xacro:property name = "base_link_ixx" value = "0.013440833333333332"/>
      <xacro:property name = "base_link_ixy" value = "0.0"/>
      <xacro:property name = "base_link_ixz" value = "0.0"/>
      <xacro:property name = "base_link_iyx" value = "0.0"/>
-     <xacro:property name = "base_link_iyy" value = "0.00276042"/>
+     <xacro:property name = "base_link_iyy" value = "0.024798337500000003"/>
      <xacro:property name = "base_link_iyz" value = "0.0"/>
      <xacro:property name = "base_link_izx" value = "0.0"/>
      <xacro:property name = "base_link_izy" value = "0.0"/>
-     <xacro:property name = "base_link_izz" value = "0.02018542"/>
+     <xacro:property name = "base_link_izz" value = "0.020185416666666664"/>
      <xacro:property name = "base_link_mass" value = "6.5"/>
      <xacro:macro name="base_link_inertial">
           <inertial>
                <mass value="${base_link_mass}" />
-               <inertia  ixx="${base_link_mass*base_link_ixx}"   ixy="${base_link_mass*base_link_ixy}"  ixz="${base_link_mass*base_link_ixz}"
+                <inertia ixx="${base_link_mass*base_link_ixx}"   ixy="${base_link_mass*base_link_ixy}"  ixz="${base_link_mass*base_link_ixz}"
+                                                                 iyy="${base_link_mass*base_link_iyy}"  iyz="${base_link_mass*base_link_iyz}"
+                                                                                                         izz="${base_link_mass*base_link_izz}"/>
+               <!-- <inertia  ixx="${base_link_mass*base_link_ixx}"   ixy="${base_link_mass*base_link_ixy}"  ixz="${base_link_mass*base_link_ixz}"
                          iyx="${base_link_mass*base_link_iyx}"   iyy="${base_link_mass*base_link_iyy}"  iyz="${base_link_mass*base_link_iyz}"
-                         izx="${base_link_mass*base_link_izx}"   izy="${base_link_mass*base_link_izy}"  izz="${base_link_mass*base_link_izz}"/>
+                         izx="${base_link_mass*base_link_izx}"   izy="${base_link_mass*base_link_izy}"  izz="${base_link_mass*base_link_izz}"/> -->
           </inertial>
      </xacro:macro>
@@ -33,6 +36,9 @@
                <mass value="${base_box_mass}"/>
                <inertia  ixx="${base_box_mass*base_box_ixx}"   ixy="${base_box_mass*base_box_ixy}"  ixz="${base_box_mass*base_box_ixz}"
+                                                               iyy="${base_box_mass*base_box_iyy}"  iyz="${base_box_mass*base_box_iyz}"
+                                                                                                    izz="${base_box_mass*base_box_izz}"  />
+               <!-- <inertia  ixx="${base_box_mass*base_box_ixx}"   ixy="${base_box_mass*base_box_ixy}"  ixz="${base_box_mass*base_box_ixz}"
                          iyx="${base_box_mass*base_box_iyx}"   iyy="${base_box_mass*base_box_iyy}"  iyz="${base_box_mass*base_box_iyz}"
-                         izx="${base_box_mass*base_box_izx}"   izy="${base_box_mass*base_box_izx}"  izz="${base_box_mass*base_box_izz}"  />
+                         izx="${base_box_mass*base_box_izx}"   izy="${base_box_mass*base_box_izx}"  izz="${base_box_mass*base_box_izz}"  />-->
           </inertial>
      </xacro:macro>

File: paxi_ws/src/paxi_description/urdf/simulation/paxi_imu_inertials.xacro (robot description, xacro)
@@ -15,6 +15,9 @@
             <mass value="${imu_hover_mass}"/>
             <inertia    ixx="${imu_hover_mass*imu_hover_ixx}"  ixy="${imu_hover_mass*imu_hover_ixy}"  ixz="${imu_hover_mass*imu_hover_ixz}"
+                                                               iyy="${imu_hover_mass*imu_hover_iyy}"  iyz="${imu_hover_mass*imu_hover_iyz}"
+                                                               izz="${imu_hover_mass*imu_hover_izz}" />
+<!--            <inertia    ixx="${imu_hover_mass*imu_hover_ixx}"  ixy="${imu_hover_mass*imu_hover_ixy}"  ixz="${imu_hover_mass*imu_hover_ixz}"
                         iyx="${imu_hover_mass*imu_hover_iyx}"  iyy="${imu_hover_mass*imu_hover_iyy}"  iyz="${imu_hover_mass*imu_hover_iyz}"
-                        izx="${imu_hover_mass*imu_hover_izx}"  izy="${imu_hover_mass*imu_hover_izy}"  izz="${imu_hover_mass*imu_hover_izz}" />
+                        izx="${imu_hover_mass*imu_hover_izx}"  izy="${imu_hover_mass*imu_hover_izy}"  izz="${imu_hover_mass*imu_hover_izz}" /> -->
         </inertial>
      </xacro:macro>

File: paxi_ws/src/paxi_description/urdf/simulation/paxi_imu_slamtec_inertials.xacro (robot description, xacro)
@@ -15,6 +15,9 @@
             <mass value="${imu_mass}" />
             <inertia    ixx="${imu_mass*imu_ixx}"   ixy="${imu_mass*imu_ixy}"  ixz="${imu_mass*imu_ixz}"
+                                                   iyy="${imu_mass*imu_iyy}"  iyz="${imu_mass*imu_iyz}"
+                                                   izz="${imu_mass*imu_izz}" />
+            <!-- <inertia    ixx="${imu_mass*imu_ixx}"   ixy="${imu_mass*imu_ixy}"  ixz="${imu_mass*imu_ixz}"
                         iyx="${imu_mass*imu_iyx}"   iyy="${imu_mass*imu_iyy}"  iyz="${imu_mass*imu_iyz}"
-                        izx="${imu_mass*imu_izx}"   izy="${imu_mass*imu_izy}"  izz="${imu_mass*imu_izz}"  />
+                        izx="${imu_mass*imu_izx}"   izy="${imu_mass*imu_izy}"  izz="${imu_mass*imu_izz}"  /> -->
         </inertial>
      </xacro:macro>

File: paxi_ws/src/paxi_description/urdf/simulation/paxi_lidar_inertials.xacro (robot description, xacro)
@@ -16,6 +16,9 @@
             <mass value="${lidar_mass}"/>
             <inertia ixx="${lidar_mass*lidar_ixx}"  ixy="${lidar_mass*lidar_ixy}"  ixz="${lidar_mass*lidar_ixz}"
+                                                    iyy="${lidar_mass*lidar_iyy}"  iyz="${lidar_mass*lidar_iyz}"
+                                                    izz="${lidar_mass*lidar_izz}"/>
+            <!-- <inertia ixx="${lidar_mass*lidar_ixx}"  ixy="${lidar_mass*lidar_ixy}"  ixz="${lidar_mass*lidar_ixz}"
                     iyx="${lidar_mass*lidar_iyx}"  iyy="${lidar_mass*lidar_iyy}"  iyz="${lidar_mass*lidar_iyz}"
-                    izx="${lidar_mass*lidar_izx}"  izy="${lidar_mass*lidar_izy}"  izz="${lidar_mass*lidar_izz}"/>
+                    izx="${lidar_mass*lidar_izx}"  izy="${lidar_mass*lidar_izy}"  izz="${lidar_mass*lidar_izz}"/> -->
         </inertial>
     </xacro:macro>
@@ -24,5 +27,5 @@
     <xacro:property name = "lidar_box_ixz" value = "0.0"/>
     <xacro:property name = "lidar_box_iyx" value = "0.0"/>
-    <xacro:property name = "lidar_box_iyy" value = "0.01408333333333333"/>
+    <xacro:property name = "lidar_box_iyy" value = "0.001408333333333333"/>
     <xacro:property name = "lidar_box_iyz" value = "0.0"/>
     <xacro:property name = "lidar_box_izx" value = "0.0"/>
@@ -34,6 +37,9 @@
             <mass value="${lidar_box_mass}" />
             <inertia ixx="${lidar_box_mass*lidar_box_ixx}"  ixy="${lidar_box_mass*lidar_box_ixy}"  ixz="${lidar_box_mass*lidar_box_ixz}"
+                                                            iyy="${lidar_box_mass*lidar_box_iyy}"  iyz="${lidar_box_mass*lidar_box_iyz}"
+                                                            izz="${lidar_box_mass*lidar_box_izz}"/>
+            <!-- <inertia ixx="${lidar_box_mass*lidar_box_ixx}"  ixy="${lidar_box_mass*lidar_box_ixy}"  ixz="${lidar_box_mass*lidar_box_ixz}"
                     iyx="${lidar_box_mass*lidar_box_iyx}"  iyy="${lidar_box_mass*lidar_box_iyy}"  iyz="${lidar_box_mass*lidar_box_iyz}"
-                    izx="${lidar_box_mass*lidar_box_izx}"  izy="${lidar_box_mass*lidar_box_izy}"  izz="${lidar_box_mass*lidar_box_izz}"/>
+                    izx="${lidar_box_mass*lidar_box_izx}"  izy="${lidar_box_mass*lidar_box_izy}"  izz="${lidar_box_mass*lidar_box_izz}"/> -->
             </inertial>
     </xacro:macro>

File: paxi_ws/src/paxi_description/urdf/simulation/paxi_wheels_inertials.xacro (robot description, xacro)
@@ -1,13 +1,13 @@
 <?xml version="1.0"?>
 <robot name="paxi_bot" xmlns:xacro="http://www.ros.org/wiki/xacro">
-    <xacro:property name = "left_wheel_ixx" value = "0.0028958333333333337"/>
+    <xacro:property name = "left_wheel_ixx" value = "0.0019723333333333333"/>
     <xacro:property name = "left_wheel_ixy" value = "0.0"/>
     <xacro:property name = "left_wheel_ixz" value = "0.0"/>
     <xacro:property name = "left_wheel_iyx" value = "0.0"/>
-    <xacro:property name = "left_wheel_iyy" value = "0.002057333333333333"/>
+    <xacro:property name = "left_wheel_iyy" value = "0.0019723333333333333"/>
     <xacro:property name = "left_wheel_iyz" value = "0.0"/>
     <xacro:property name = "left_wheel_izx" value = "0.0"/>
     <xacro:property name = "left_wheel_izy" value = "0.0"/>
-    <xacro:property name = "left_wheel_izz" value = "0.0036979999999999995"/>
+    <xacro:property name = "left_wheel_izz" value = "0.0035280000000000003"/>
     <!-- ref: https://www.parallax.com/product/6-5-hub-motor-with-encoder/ -->
     <xacro:property name = "left_wheel_mass" value = "3.1"/>
@@ -15,18 +15,21 @@
         <inertial>
             <mass value="${left_wheel_mass}" />
-            <inertia    ixx="${left_wheel_mass*left_wheel_ixx}"   ixy="${left_wheel_mass*left_wheel_ixy}"  ixz="${left_wheel_mass*left_wheel_ixz}"
+            <inertia ixx="${left_wheel_mass*left_wheel_ixx}"    ixy="${left_wheel_mass*left_wheel_ixy}"  ixz="${left_wheel_mass*left_wheel_ixz}"
+                                                                iyy="${left_wheel_mass*left_wheel_iyy}"  iyz="${left_wheel_mass*left_wheel_iyz}"
+                                                                izz="${left_wheel_mass*left_wheel_izz}"  />
+            <!-- <inertia    ixx="${left_wheel_mass*left_wheel_ixx}"   ixy="${left_wheel_mass*left_wheel_ixy}"  ixz="${left_wheel_mass*left_wheel_ixz}"
                         iyx="${left_wheel_mass*left_wheel_iyx}"   iyy="${left_wheel_mass*left_wheel_iyy}"  iyz="${left_wheel_mass*left_wheel_iyz}"
-                        izx="${left_wheel_mass*left_wheel_izx}"   izy="${left_wheel_mass*left_wheel_izy}"  izz="${left_wheel_mass*left_wheel_izz}"  />
+                        izx="${left_wheel_mass*left_wheel_izx}"   izy="${left_wheel_mass*left_wheel_izy}"  izz="${left_wheel_mass*left_wheel_izz}"  /> -->
         </inertial>
     </xacro:macro>
-    <xacro:property name = "right_wheel_ixx" value = "0.0028958333333333337"/>
+    <xacro:property name = "right_wheel_ixx" value = "0.0019723333333333333"/>
     <xacro:property name = "right_wheel_ixy" value = "0.0"/>
     <xacro:property name = "right_wheel_ixz" value = "0.0"/>
     <xacro:property name = "right_wheel_iyx" value = "0.0"/>
-    <xacro:property name = "right_wheel_iyy" value = "0.002057333333333333"/>
+    <xacro:property name = "right_wheel_iyy" value = "0.0019723333333333333"/>
     <xacro:property name = "right_wheel_iyz" value = "0.0"/>
     <xacro:property name = "right_wheel_izx" value = "0.0"/>
     <xacro:property name = "right_wheel_izy" value = "0.0"/>
-    <xacro:property name = "right_wheel_izz" value = "0.0036979999999999995"/>
+    <xacro:property name = "right_wheel_izz" value = "0.0035280000000000003"/>
     <!-- ref: https://www.parallax.com/product/6-5-hub-motor-with-encoder/ -->
     <xacro:property name = "right_wheel_mass" value = "3.1"/>
@@ -34,7 +37,10 @@
         <inertial>
             <mass value="${right_wheel_mass}" />
-            <inertia    ixx="${right_wheel_mass*right_wheel_ixx}"   ixy="${right_wheel_mass*right_wheel_ixy}"  ixz="${right_wheel_mass*right_wheel_ixz}"
+            <inertia    ixx="${right_wheel_mass*right_wheel_ixx}"   ixy="${right_wheel_mass*right_wheel_ixy}"   ixz="${right_wheel_mass*right_wheel_ixz}"
+                                                                    iyy="${right_wheel_mass*right_wheel_iyy}"   iyz="${right_wheel_mass*right_wheel_iyz}"
+                                                                                                                izz="${right_wheel_mass*right_wheel_izz}"  />
+            <!-- <inertia    ixx="${right_wheel_mass*right_wheel_ixx}"   ixy="${right_wheel_mass*right_wheel_ixy}"  ixz="${right_wheel_mass*right_wheel_ixz}"
                         iyx="${right_wheel_mass*right_wheel_iyx}"   iyy="${right_wheel_mass*right_wheel_iyy}"  iyz="${right_wheel_mass*right_wheel_iyz}"
-                        izx="${right_wheel_mass*right_wheel_izx}"   izy="${right_wheel_mass*right_wheel_izy}"  izz="${right_wheel_mass*right_wheel_izz}"  />
+                        izx="${right_wheel_mass*right_wheel_izx}"   izy="${right_wheel_mass*right_wheel_izy}"  izz="${right_wheel_mass*right_wheel_izz}"  /> -->
         </inertial>
     </xacro:macro>
@@ -52,7 +58,10 @@
          <inertial>
             <mass value="${caster_wheel_mass}" />
-            <inertia    ixx="${caster_wheel_mass*caster_wheel_ixx}"   ixy="${caster_wheel_mass*caster_wheel_ixy}"  ixz="${caster_wheel_mass*caster_wheel_ixz}"
+            <inertia ixx="${caster_wheel_mass*caster_wheel_ixx}"   ixy="${caster_wheel_mass*caster_wheel_ixy}"     ixz="${caster_wheel_mass*caster_wheel_ixz}"
+                                                                    iyy="${caster_wheel_mass*caster_wheel_iyy}"     iyz="${caster_wheel_mass*caster_wheel_iyz}"
+                                                                                                                    izz="${caster_wheel_mass*caster_wheel_izz}"  />
+             <!-- <inertia    ixx="${caster_wheel_mass*caster_wheel_ixx}"   ixy="${caster_wheel_mass*caster_wheel_ixy}"  ixz="${caster_wheel_mass*caster_wheel_ixz}"
                         iyx="${caster_wheel_mass*caster_wheel_iyx}"   iyy="${caster_wheel_mass*caster_wheel_iyy}"  iyz="${caster_wheel_mass*caster_wheel_iyz}"
-                        izx="${caster_wheel_mass*caster_wheel_izx}"   izy="${caster_wheel_mass*caster_wheel_izy}"  izz="${caster_wheel_mass*caster_wheel_izz}"  />
+                        izx="${caster_wheel_mass*caster_wheel_izx}"   izy="${caster_wheel_mass*caster_wheel_izy}"  izz="${caster_wheel_mass*caster_wheel_izz}"  />  -->
         </inertial>
     </xacro:macro>
